File: st77xx.kicad_sch (KiCad schematic)
At the start: 8 parts, among them J1 Pins, J2 Flex, Q1 S8050, U1 XC6206PxxxMR

Commit message: Fix schematic
Connections:
- net CS: now also R3.1; no longer R3.2
- net GND: now also R3.2; no longer R3.1
Other:
- moved on the sheet: J1, J2, Q1, R2, U1

Commit message: Update
Parts:
- removed J2: Flex, symbol Connector_Generic:Conn_01x12
- removed Q1: S8050, Package_TO_SOT_THT:TO-92_Inline, symbol Transistor_BJT:S8050
- removed R1: 5, symbol Device:R
- removed R2: 2k2, symbol Device:R
- removed R3: 50k, symbol Device:R
- removed R4: 10k, symbol Device:R
- added C1: 100n, Capacitor_SMD:C_0603_1608Metric, symbol Device:C_Small
- added C2, C3: 1u, Capacitor_SMD:C_0603_1608Metric, symbol Device:C_Small
- added DS1: ST77xx_FPC_12pin, ST77xx_FPC:ST77XX_FPC_12pin_0.8mm_Solder, symbol ST77xx_FPC:ST77xx_FPC_12pin
- added Q1: SS8050, Package_TO_SOT_SMD:SOT-23, symbol Transistor_BJT:SS8050
- added R1, R2, R3: 50k, Resistor_SMD:R_0603_1608Metric, symbol Device:R_Small
- added R4: 2k2, Resistor_SMD:R_0603_1608Metric, symbol Device:R_Small
- J1: footprint (none) -> Connector_PinHeader_2.54mm:PinHeader_1x08_P2.54mm_Vertical
Connections:
- net +3.3V: now also C1.1, C2.1, DS1.3 (LEDA), DS1.4 (VDD), R1.1
- net BLK: now also R4.1
- net CS: now also DS1.8 (C/S), R2.1
- net DC: now also DS1.7 (D/C)
- net GND: now also C1.2, C2.2, C3.2, DS1.1 (GND), DS1.12 (GND), DS1.5 (GND), DS1.6 (GND), Q1.2 (E), R2.2
- net RES: now also DS1.11 (RESET), R1.2
- net SCL: now also DS1.9 (SCL)
- net SDA: now also DS1.10 (SDA)
- net VCC: now also C3.1
- new net: DS1.2 (LEDK), R3.1
- new net: Q1.1 (B), R4.2
- new net: Q1.3 (C), R3.2
- no-connect marks 1 -> 0
Other:
- note added: "3.3V regulator when VCC > 3.3V"
- note added: "CS pull-down"
- note added: "LED return path Enabled by BLK high"
- note added: "May be replaced with N-FET"
- note added: "RES pull-up"
- moved on the sheet: U1

Commit message: Fix LEDK resistor
Parts:
- R3: value 50k -> 30R
Changed lines of the file:
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@@
 			)
 		)
-		(property "Value" "50k"
+		(property "Value" "30R"
 			(at 182.88 115.5699 0)
 			(effects
